Commit message: cobot

File: cobot_description/urdf/abb_vibrategripper.xacro (robot description, xacro)
@@ -3,12 +3,9 @@
   <xacro:include filename="$(find irb120_description)/urdf/irb120.xacro"/>
   <xacro:abb_irb120 prefix=""/>
-  <xacro:include filename="$(find robotiq_3f_description)/urdf/robotiq-3f-gripper_articulated.xacro"  />
-	<xacro:property name="PI" value="3.1415926535897931"/>
- <!-- verificar angulo de support_gripper -->
-  <link name="gripper_support_link">
+  <link name="vibration_gripper">
     <inertial>
       <origin
         xyz="0 0 0"
-        rpy="1.570796327 0 0" />
+        rpy="0 0 0" />
       <mass
         value="0.30915" />
@@ -23,9 +20,9 @@
     <visual>
       <origin
-        xyz="0 0 0"
-        rpy="1.570796327 0 0.523598" />
+        xyz="0.0695 -0.031 0"
+        rpy="-1.570796327 0 1.570796327" />
       <geometry>
         <mesh
-          filename="package://irb120_description/meshes/supports/support_gripper.stl" />
+          filename="package://cobot_description/meshes/GRIPER_BELTm.stl" />
       </geometry>
       <material name="green"/>
@@ -33,30 +30,25 @@
     <collision>
       <origin
-        xyz="0 0 0"
-        rpy="1.570796327 0 0.523598" />
+        xyz="0.0695 -0.031 0"
+        rpy="-1.570796327 0 1.570796327" />
       <geometry>
         <mesh
-          filename="package://irb120_description/meshes/supports/support_gripper.stl" />
+          filename="package://cobot_description/meshes/GRIPER_BELTm.stl" />
       </geometry>
     </collision>
   </link>
-  <joint name="irb120_joint_gripper_support" type="fixed">
+  <joint name="gripper" type="fixed">
     <parent link="tool0"/>
-    <child link="gripper_support_link"/>
-    <origin rpy="0 0 0" xyz="0 0 0.008"/>
-  </joint>
-  <joint name="irb120_support_gripper" type="fixed">
-    <parent link="gripper_support_link"/>
-    <child link="palm"/>
-    <origin rpy="${PI/2} 0 0" xyz="0 0 0.05"/>
+    <child link="vibration_gripper"/>
+    <origin rpy="0 0 0" xyz="0 0 0.1908"/>s
   </joint>
   <!-- end effect point -->
-  <joint name="end_effect_point3f" type="fixed">
-    <origin rpy="0 0 0" xyz="0 0 0.15"/>
-    <parent link="gripper_support_link"/>
-    <child link="end_effect_point3f"/>
+  <joint name="end_eff_point_vibrationgripper" type="fixed">
+    <origin rpy="0 0 0" xyz="-0.12 0.025 0.172"/>
+    <parent link="tool0"/>
+    <child link="end_eff_point_vibrationgripper"/>
   </joint>
   <!-- end effect point -->
-  <link name="end_effect_point3f">
+  <link name="end_eff_point_vibrationgripper">
     <visual>
       <origin rpy="0 0 0" xyz="0 0 0"/>

File: cobot_description/urdf/cobot_main.xacro (robot description, xacro)
@@ -3,4 +3,4 @@
   <xacro:include filename="$(find cobot_description)/urdf/table.xacro"/>
   <xacro:include filename="$(find cobot_description)/urdf/indy7_gripper2f.xacro"/>
-  <xacro:include filename="$(find cobot_description)/urdf/abb_gripper3f.xacro"/>
+  <xacro:include filename="$(find cobot_description)/urdf/abb_vibrategripper.xacro"/>
 </robot>

File: cobot_description/urdf/indy7_gripper2f.xacro (robot description, xacro)
@@ -27,5 +27,5 @@
       <origin
         xyz="0 0 0"
-        rpy="1.570796327 0 0" />
+        rpy="0 0 0" />
       <mass
         value="0.30915" />
@@ -40,9 +40,9 @@
     <visual>
       <origin
-        xyz="0 0 0"
-        rpy="1.570796327 0 0.523598" />
+        xyz="-0.045 -0.045 -0.022"
+        rpy="0 0 0" />
       <geometry>
         <mesh
-          filename="package://indy7_description/meshes/supports/support_gripper.stl" />
+          filename="package://indy7_description/meshes/supports/indy7_to_irb120_TCP.stl" />
       </geometry>
       <material name="green"/>
@@ -50,9 +50,9 @@
     <collision>
       <origin
-        xyz="0 0 0"
-        rpy="1.570796327 0 0.523598" />
+        xyz="-0.045 -0.045 -0.022"
+        rpy="0 0 0" />
       <geometry>
         <mesh
-          filename="package://indy7_description/meshes/supports/support_gripper.stl" />
+          filename="package://indy7_description/meshes/supports/indy7_to_irb120_TCP.stl" />
       </geometry>
     </collision>
@@ -61,19 +61,19 @@
     <parent link="tcp"/>
     <child link="support_gripper_link"/>
-    <origin rpy="0 0 0" xyz="0 0 0.008"/>
+    <origin rpy="0 0 0" xyz="0 0 0.02"/>
   </joint>
   <joint name="indy7_support_gripper" type="fixed">
     <parent link="support_gripper_link"/>
     <child link="coupling_link"/>
-    <origin rpy="0 0 ${PI/2}" xyz="0 0 0"/>
+    <origin rpy="0 0 ${PI/2}" xyz="0 0 -0.003"/>
   </joint>
   <!-- end effect point -->
-  <joint name="end_effect_point" type="fixed">
-    <origin rpy="0 0 0" xyz="0 0 0.17"/>
+  <joint name="end_eff_point_2f" type="fixed">
+    <origin rpy="0 0 0" xyz="0 0 0.23"/>
     <parent link="tcp"/>
-    <child link="end_effect_point"/>
+    <child link="end_eff_point_2f"/>
   </joint>
   <!-- end effect point -->
-  <link name="end_effect_point">
+  <link name="end_eff_point_2f">
     <visual>
       <origin rpy="0 0 0" xyz="0 0 0"/>

File: cobot_description/urdf/table.xacro (robot description, xacro)
@@ -25,10 +25,12 @@
 		<parent link="table"/>
 		<child link="support_indy7"/>
-		<origin xyz="-0.7 0 0" rpy="0 0 0"/>
+		<origin xyz="-0.65 0.0125 0" rpy="0 0 0"/>
+		<!-- <origin xyz="-0.65 0.0125 0" rpy="0 0 0"/> -->
 	</joint>
 	<joint name="abb" type="fixed">
 		<parent link="table"/>
 		<child link="base_link"/>
-		<origin xyz="0.7 0 0" rpy="0 0 3.1416"/>
+		<origin xyz="0.64 0 0" rpy="0 0 3.1416"/>
+		<!-- <origin xyz="0.7 0 0" rpy="0 0 3.1416"/> -->
 	</joint>
 </robot>

Commit message: update

File: cobot_description/urdf/abb_vibrategripper.xacro (robot description, xacro)
@@ -45,5 +45,7 @@
   <!-- end effect point -->
   <joint name="end_eff_point_vibrationgripper" type="fixed">
-    <origin rpy="0 0 0" xyz="-0.12 0.025 0.172"/>
+    <!-- <origin rpy="0 0 0" xyz="-0.12 0.025 0.172"/> -->
+    <origin rpy="0 0 0" xyz="-0.12 0.025 0.1855"/>
+    <!-- <origin rpy="0 0 0" xyz="-0.12 0.025 0.1855"/> -->
     <parent link="tool0"/>
     <child link="end_eff_point_vibrationgripper"/>

File: cobot_description/urdf/cobot.urdf (robot description, URDF)
Before this commit: robot cobot, 39 links, 38 joints
Links:
- removed link base
- removed link gripper_support_link
- link support_gripper_link: geometry collision mesh filename=package://indy7_description/meshes/supports/indy7_to_irb120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; visual mesh filename=package://indy7_description/meshes/supports/indy7_to_irb120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
- link vibration_gripper: geometry collision mesh filename=package://cobot_description/meshes/GRIPER_BELTm.stl; visual mesh filename=package://cobot_description/meshes/GRIPER_BELTm.stl
Joints:
- removed joint base_link-base
- removed joint irb120_joint_gripper_support
- joint abb: origin xyz=0.7 0 0 rpy=0 0 3.1416 -> xyz=0.64 0 0 rpy=0 0 3.1416
- joint end_eff_point_2f: origin xyz=0 0 0.17 rpy=0 0 0 -> xyz=0 0 0.23 rpy=0 0 0
- joint end_eff_point_vibrationgripper: origin xyz=-0.09 0.02 0.15 rpy=0 0 0 -> xyz=-0.12 0.025 0.1855 rpy=0 0 0
- joint gripper: origin xyz=0 0 0.05 rpy=0 0 0 -> xyz=0 0 0.1908 rpy=0 0 0; parent gripper_support_link -> tool0
- joint indy7: origin xyz=-0.7 0 0 rpy=0 0 0 -> xyz=-0.65 0.0125 0 rpy=0 0 0
- joint indy7_joint_tcp: origin xyz=0 0 0.008 rpy=0 0 0 -> xyz=0 0 0.02 rpy=0 0 0
- joint indy7_support_gripper: origin xyz=0 0 0 rpy=0 0 1.57079632679 -> xyz=0 0 -0.003 rpy=0 0 1.57079632679
- joint joint_6: limit lower=-6.98132 upper=6.98132 effort=0 velocity=7.33038 -> lower=-3.98132 upper=3.98132 effort=0 velocity=7.33038
